Commit message: deadlock

File: examples/urdfs/cup/cup_green.urdf (robot description, URDF)
Before this commit: robot cube.urdf, 1 links, 0 joints
Links:
- link baseLink: geometry visual mesh filename=textured-0008192.obj scale=0.5 0.5 0.5

File: examples/urdfs/cup/cup_red.urdf (robot description, URDF)
Before this commit: robot cube.urdf, 1 links, 0 joints
Links:
- link baseLink: geometry visual mesh filename=textured-0008192.obj scale=0.5 0.5 0.5
