Commit message: fixed multirobot

File: examples/urdfs/dinova/dinova.urdf (robot description, URDF)
Before this commit: robot dingo_kinova, 30 links, 29 joints
Joints:
- joint arm_tool_frame_joint: origin xyz=0 0 0.08 rpy=0 0 0 -> xyz=0 0 0.12 rpy=0 0 0

Commit message: end-goal now changed to the tool-frame everywhere instead of end-effector frame.

File: examples/urdfs/dinova/dinova.urdf (robot description, URDF)
Before this commit: robot dingo_kinova, 30 links, 29 joints
Joints:
- joint arm_tool_frame_joint: origin xyz=0 0 0.12 rpy=0 0 0 -> xyz=0 0 0.14 rpy=0 0 0

Commit message: bug found, rollouts don't work well, going back in versions.

File: examples/urdfs/dinova/dinova.urdf (robot description, URDF)
Before this commit: robot dingo_kinova, 30 links, 29 joints
Joints:
- joint arm_tool_frame_joint: origin xyz=0 0 0.14 rpy=0 0 0 -> xyz=0 0 0.12 rpy=0 0 0

Commit message: fabrics example, have to fix gomp

File: examples/urdfs/dinova/dinova.urdf (robot description, URDF)
Before this commit: robot dingo_kinova, 30 links, 29 joints
Joints:
- joint arm_tool_frame_joint: origin xyz=0 0 0.12 rpy=0 0 0 -> xyz=0 0 0.08 rpy=0 0 0
