Commit message: fixing obstacles, metrics,...

File: examples/urdfs/dinova/dinova_1.urdf (robot description, URDF)
Before this commit: robot dingo_kinova, 30 links, 29 joints
Joints:
- joint arm_tool_frame_joint: origin xyz=0 0 0.08 rpy=0 0 0 -> xyz=0 0 0.13 rpy=0 0 0

File: examples/urdfs/dinova/dinova_2.urdf (robot description, URDF)
Before this commit: robot dingo_kinova, 30 links, 29 joints
Joints:
- joint arm_tool_frame_joint: origin xyz=0 0 0.08 rpy=0 0 0 -> xyz=0 0 0.13 rpy=0 0 0

File: examples/urdfs/dinova/dinova_3.urdf (robot description, URDF)
Before this commit: robot dingo_kinova, 30 links, 29 joints
Joints:
- joint arm_tool_frame_joint: origin xyz=0 0 0.08 rpy=0 0 0 -> xyz=0 0 0.13 rpy=0 0 0

File: examples/urdfs/dinova/dinova_4.urdf (robot description, URDF)
Before this commit: robot dingo_kinova, 30 links, 29 joints
Joints:
- joint arm_tool_frame_joint: origin xyz=0 0 0.08 rpy=0 0 0 -> xyz=0 0 0.13 rpy=0 0 0
