Commit message: working example of tworobots_withoutobstacle, plus separate rollout controller

File: examples/urdfs/table_100x100/table_square.urdf (robot description, URDF)
Before this commit: robot urdf_table, 2 links, 1 joints
Links:
- link baseLink: geometry collision box size=1 1 0.02; visual box size=0.025 0.025 0.30

File: examples/urdfs/table_50x50/table_square.urdf (robot description, URDF)
Before this commit: robot urdf_table, 2 links, 1 joints
Links:
- link baseLink: geometry collision box size=0.5 0.5 0.02; visual box size=0.025 0.025 0.30
